File: TPS63021.kicad_sch (KiCad schematic)
At the start: 13 parts, among them U3 TPS63021DSJR

Commit message: add footprint 18650 batteryClip
Connections:
- net +3.3V renamed V_{OUT}3.3V
- net VOUT renamed V_{IN}
Changed lines of the file:
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@@
 		)
 	)
-	(label "VOUT"
+	(hierarchical_label "V_{OUT}3.3V"
+		(shape output)
+		(at 238.76 78.74 0)
+		(fields_autoplaced yes)
+		(effects
+			(font
+				(size 1.27 1.27)
+			)
+			(justify left)
+		)
+	)
+	(hierarchical_label "V_{IN}"
+		(shape input)
 		(at 87.63 78.74 180)
 		(fields_autoplaced yes)
@@
 				(size 1.27 1.27)
 			)
-			(justify right bottom)
+			(justify right)
 		)
 	)
@@
 					(unit 1)
 				)
-			)
-		)
-	)
-	(symbol
-		(lib_id "power:+3.3V")
-		(at 238.76 78.74 270)
-		(unit 1)
-		(exclude_from_sim no)
-		(in_bom yes)
-		(on_board yes)
-		(dnp no)
-		(property "Reference" "#PWR041"
-			(at 234.95 78.74 0)
-			(effects
-				(font
-					(size 1.27 1.27)
-				)
-				(hide yes)
-			)
-		)
-		(property "Value" "+3.3V"
-			(at 243.332 78.486 90)
-			(effects
-				(font
-					(size 1.27 1.27)
-				)
-				(justify left)
-			)
-		)
-		(property "Footprint" ""
-			(at 238.76 78.74 0)
-			(effects
-				(font
-					(size 1.27 1.27)
-				)
-				(hide yes)
-			)
-		)
-		(property "Datasheet" ""
-			(at 238.76 78.74 0)
-			(effects
-				(font
-					(size 1.27 1.27)
-				)
-				(hide yes)
-			)
-		)
-		(property "Description" "Power symbol creates a global label with name \"+3.3V\""
-			(at 238.76 78.74 0)
-			(effects
-				(font
-					(size 1.27 1.27)
-				)
-				(hide yes)
-			)
-		)
-		(pin "1"
-		)
-		(instances
-			(project "Template"
-				(path "/251827e7-9515-4eb7-984d-8b86837d4b30/c43323f0-476e-4b9f-92da-cf6d01a9204e"
-					(reference "#PWR041")
-					(unit 1)
-				)
